File: hardware/CybICS/CybICS.kicad_sch (KiCad schematic)
At the start: 16 parts, among them J1 Raspberry_Pi_2_3, U1 STM32G070RBTx

Commit message: Further development of the schematic and pcb
Parts:
- added C1, C2, C4: 100nF, Capacitor_SMD:C_0805_2012Metric_Pad1.18x1.45mm_HandSolder, symbol Device:C
- added C3: 4.7μF, Capacitor_SMD:C_0805_2012Metric_Pad1.18x1.45mm_HandSolder, symbol Device:C
- added D11, D12: LED GREEN, LED_SMD:LED_1210_3225Metric_Pad1.42x2.65mm_HandSolder, symbol Device:LED
- added H1, H2, H3, H4: MountingHole, MountingHole:MountingHole_3.2mm_M3, symbol Mechanical:MountingHole
- added R1, R10, R11, R12, R2, R3, R4, R5, R6, R7, R8, R9: 1000R, Resistor_SMD:R_0805_2012Metric_Pad1.20x1.40mm_HandSolder, symbol Device:R
- added R13, R14, R15, R16, R17: 0R, Resistor_SMD:R_0805_2012Metric_Pad1.20x1.40mm_HandSolder, symbol Device:R
- added RV1: R_Potentiometer, Potentiometer_SMD:Potentiometer_Bourns_3314J_Vertical, symbol Device:R_Potentiometer
- added SW1: SW_Push, Button_Switch_SMD:SW_Push_1P1T_NO_6x6mm_H9.5mm, symbol Switch:SW_Push
Connections:
- net at D5.1 (K): now also R10.2
- net +3V3: now reaches D5.2 (A)
- net +3V3: now also D1.2 (A), D10.2 (A), D2.2 (A), D3.2 (A), D4.2 (A), D6.2 (A), D7.2 (A), D8.2 (A), D9.2 (A), DS1.15 (LED(+)), DS1.2 (VDD), J1.1 (3V3), J1.17 (3V3), U1.7 (VREF+), U1.8 (VDD), C1.1, C2.1, C3.1, D11.2 (A), D12.2 (A), RV1.3
- net at D2.1 (K): now also R7.2
- net at D3.1 (K): now also R8.2
- net at D7.1 (K): now also R2.2
- net GND: now reaches DS1.1 (VSS)
- net GND: now also DS1.16 (LED(-)), DS1.5 (R/W), J1.14 (GND), J1.20 (GND), J1.25 (GND), J1.30 (GND), J1.34 (GND), J1.39 (GND), J1.6 (GND), J1.9 (GND), U1.9 (VSS), C1.2, C2.2, C3.2, C4.2, RV1.1, SW1.1
- net at DS1.3 (VO): now also RV1.2
- net D_rs: now reaches DS1.4 (RS)
- net D_enable: now reaches DS1.6 (E)
- net at D6.1 (K): now also R1.2
- net at D9.1 (K): now also R4.2
- net at D1.1 (K): now also R6.2
- net at D8.1 (K): now also R3.2
- net at J1.12 (GPIO18/PWM0): now also R13.2
- net at J1.18 (GPIO24): now also R14.2
- net at J1.22 (GPIO25): now also R15.2
- net at J1.3 (SDA/GPIO2): now also R16.1
- net at J1.5 (SCL/GPIO3): now also R17.1
- net STMnrst: now reaches U1.12 (NRST)
- net STMnrst: now also C4.1, R13.1, SW1.2
- net USART1_TX: now reaches U1.37 (PA9/NC)
- net USART1_RX: now reaches U1.42 (PA10/NC)
- net SWDIO: now reaches U1.45 (PA13)
- net SWDIO: now also R14.1
- net SWCLK: now reaches U1.46 (PA14)
- net SWCLK: now also R15.1
- net I2C1_SDA: now reaches U1.61 (PB7)
- net I2C1_SDA: now also R16.2
- net I2C1_SCL: now reaches U1.62 (PB8)
- net I2C1_SCL: now also R17.2
- net at D4.1 (K): now also R9.2
- net at D10.1 (K): now also R5.2
- new net: D11.1 (K), R11.2
- new net: D12.1 (K), R12.2
Other:
- note added: "STM32G070RBT6"
- moved on the sheet: D1, D10, D2, D3, D4, D5, D6, D7, D8, D9, DS1, J1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

Commit message: further development
Parts:
- added D13, D15, D17, D19: LED GREEN, LED_SMD:LED_1210_3225Metric_Pad1.42x2.65mm_HandSolder, symbol Device:LED
- added D14, D16, D18: LED RED, LED_SMD:LED_1210_3225Metric_Pad1.42x2.65mm_HandSolder, symbol Device:LED
- added J2: Conn_01x03_Pin, Connector_PinHeader_2.54mm:PinHeader_1x03_P2.54mm_Vertical, symbol Connector:Conn_01x03_Pin
- added J3: Conn_01x05_Pin, Connector_PinHeader_2.54mm:PinHeader_1x05_P2.54mm_Vertical, symbol Connector:Conn_01x05_Pin
- added R18, R19: 0R, Resistor_SMD:R_0805_2012Metric_Pad1.20x1.40mm_HandSolder, symbol Device:R
- added R20, R21, R22, R23, R24, R25, R26: 100R, Resistor_SMD:R_0805_2012Metric_Pad1.20x1.40mm_HandSolder, symbol Device:R
- added R27: 1kR, Resistor_SMD:R_0805_2012Metric_Pad1.20x1.40mm_HandSolder, symbol Device:R
- added SW2: SW_Push, Button_Switch_THT:SW_PUSH_6mm_H5mm, symbol Switch:SW_Push
- R1, R10, R11, R12, R2, R3, R4, R5, R6, R7, R8, R9: value 1000R -> 100R
- SW1: footprint Button_Switch_SMD:SW_Push_1P1T_NO_6x6mm_H9.5mm -> Button_Switch_THT:SW_PUSH_6mm_H5mm
Connections:
- net +3V3: now also D13.2 (A), D14.2 (A), D15.2 (A), D16.2 (A), D17.2 (A), D18.2 (A), D19.2 (A), J3.1 (Pin_1), R27.1
- net D_enable: now also U1.30 (PB10)
- net D_rs: now also U1.31 (PB11)
- net GND: now also J2.3 (Pin_3), J3.5 (Pin_5), R20.1
- net STMnrst: now also J3.4 (Pin_4)
- net SWCLK: now also J3.3 (Pin_3)
- net SWDIO: now also J3.2 (Pin_2)
- net USART1_RX: now also J2.1 (Pin_1), R18.1
- net USART1_TX: now also J2.2 (Pin_2), R19.1
- net PD6: now reaches R1.1
- net PD6: now also U1.56 (PD6)
- net PD5: now reaches R2.1
- net PD5: now also U1.55 (PD5)
- net PD2: now reaches R5.1
- net PD2: now also U1.52 (PD2)
- net PB3: now reaches R10.1
- net PB3: now also U1.57 (PB3)
- net D_d4: now reaches DS1.11 (D4)
- net D_d4: now also U1.32 (PB12)
- net D_d5: now reaches DS1.12 (D5)
- net D_d5: now also U1.33 (PB13)
- net D_d6: now reaches DS1.13 (D6)
- net D_d6: now also U1.34 (PB14)
- net D_d7: now reaches DS1.14 (D7)
- net D_d7: now also U1.35 (PB15)
- net PB9: now reaches R8.1
- net PB9: now also U1.63 (PB9)
- net PD4: now reaches R3.1
- net PD4: now also U1.54 (PD4)
- net PD3: now reaches R4.1
- net PD3: now also U1.53 (PD3)
- net at J1.10 (GPIO15/RXD): now also R19.2
- net at J1.8 (GPIO14/TXD): now also R18.2
- net PB6: now reaches R7.1
- net PB6: now also U1.60 (PB6)
- net PB4: now reaches U1.58 (PB4)
- net PB4: now also R9.1
- net PB5: now reaches U1.59 (PB5)
- net PB5: now also R6.1
- net PC10: now reaches U1.64 (PC10)
- net PC10: now also SW2.1
- new net: D18.1 (K), R25.2
- new net: D16.1 (K), R23.2
- new net: D19.1 (K), R26.2
- new net: R27.2, SW2.2
- new net: D17.1 (K), R24.2
- new net: D14.1 (K), R21.2
- new net: D13.1 (K), R20.2
- new net: D15.1 (K), R22.2
Other:
- note added: "Blowout"
- note added: "SWD"
- note added: "System"
- note added: "System Valve"
- note added: "UART"
- moved on the sheet: FID1, FID2, FID3, H1, H2, H3, H4, R13, R14, R15

Commit message: Update on schematic and PCB
Parts:
- removed H4: MountingHole, MountingHole:MountingHole_3.2mm_M3, symbol Mechanical:MountingHole
- DS1: value WC1602A / HD44780 -> WC1602A/HD44780
Connections:
- net PA12: now reaches R25.1
- net PA12: now also U1.44 (PA12/PA10)
- net ST_heartbeat: now reaches R11.1
- net ST_heartbeat: now also U1.16 (PC3)
- net PC8: now reaches R23.1
- net PC8: now also U1.48 (PC8)
- net PC9: now reaches R24.1
- net PC9: now also U1.49 (PC9)
- net PD1: now reaches R21.1
- net PD1: now also U1.51 (PD1)
- net PA0: now reaches J1.24 (~{CE0}/GPIO8)
- net PA0: now also U1.17 (PA0)
- net PA1: now reaches J1.26 (~{CE1}/GPIO7)
- net PA1: now also U1.18 (PA1)
- net PA2: now reaches J1.28 (ID_SC/GPIO1)
- net PA2: now also U1.19 (PA2)
- net PA3: now reaches J1.32 (PWM0/GPIO12)
- net PA3: now also U1.20 (PA3)
- net PA4: now reaches J1.36 (GPIO16)
- net PA4: now also U1.21 (PA4)
- net PA5: now reaches J1.38 (GPIO20/MOSI1)
- net PA5: now also U1.22 (PA5)
- net PA6: now reaches J1.40 (GPIO21/SCLK1)
- net PA6: now also U1.23 (PA6)
- net RP_heartbeat: now reaches J1.7 (GCLK0/GPIO4)
- net RP_heartbeat: now also R12.1
- net PA15: now reaches R26.1
- net PA15: now also U1.47 (PA15)
- net PD0: now reaches R22.1
- net PD0: now also U1.50 (PD0)
- no-connect marks 0 -> 42
Other:
- note added: "Button"
- note added: "Display HD44780"
- note added: "Raspberry Pi"
- moved on the sheet: D10, D11, D12, D13, D6, D7, D8, D9, J2, J3, R1, R11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
