File: hardware/CybICS.kicad_pcb (KiCad board)
At the start: 2 copper layers, 160 x 100 mm, 65 parts, among them J1 Raspberry_Pi_2_3, J2 Conn_01x03_Pin, J3 Conn_01x05_Pin, SW1 SW_Push, SW2 SW_Push, U1 STM32G070RBTx

Commit message: Added remote debugging from dev computer to rpi to stm32
Connections:
- DS1 pad 2: +3V3 -> +5V
- J1 pad 2: unconnected-(J1-5V-Pad2) -> +5V
- J1 pad 4: unconnected-(J1-5V-Pad4) -> +5V
Routing:
- net +5V: track 0.00 -> 80.6 mm

Commit message: Updated hardware
Parts:
- removed the REF** at (70.8, 58.8)
- added R28: 10kR, Resistor_SMD:R_0805_2012Metric_Pad1.20x1.40mm_HandSolder, F.Cu at (64.8, 99.4)
- added REF**: OSHW-Logo2_7.3x6mm_Copper, Symbol:OSHW-Logo2_7.3x6mm_Copper, F.Cu at (69.8, 56.8)
- J1: footprint Connector_PinHeader_2.54mm:PinHeader_2x20_P2.54mm_Vertical -> Module:Raspberry_Pi_Zero_Socketed_THT_FaceDown_MountingHoles; moved to B.Cu
- moved J1 17.8 mm to (70.9, 125.5), turned to -90 degrees
- moved R13 17.3 mm to (86.8, 118.5)
- moved R14 17.3 mm to (90.8, 118.5)
- moved R16 17.3 mm to (70.8, 118.5)
- moved R17 17.3 mm to (74.8, 118.5)
- moved R18 17.3 mm to (78.8, 118.5)
- moved R19 17.3 mm to (82.8, 118.5)
- moved R15 17.3 mm to (94.5, 118.5)
- moved C2 14.3 mm to (84.8, 102.6)
- moved C1 14.3 mm to (84.8, 107.3)
- moved C3 14.3 mm to (81.5, 107.3)
- moved C4 14.3 mm to (83.3, 111.6)
- moved J2 14.3 mm to (111.8, 110.6)
- moved J3 14.3 mm to (68.8, 110.7)
- moved R21 14.3 mm to (117.8, 91.6)
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Routing:
- net /STMnrst: track 49.0 -> 70.0 mm, vias 0 -> 2
- net /PC10: track 56.3 -> 39.5 mm
- net /RP_heartbeat: track 31.5 -> 19.9 mm
- net /ST_heartbeat: track 28.5 -> 36.9 mm
- net Net-(D18-K): track 73.5 -> 66.6 mm
- net /D_enable: track 65.5 -> 58.6 mm
- net Net-(D19-K): track 70.6 -> 63.8 mm
- net Net-(D17-K): track 86.4 -> 79.6 mm
- net Net-(D16-K): track 85.9 -> 79.3 mm
- net /D_d5: track 76.6 -> 70.5 mm, vias 2 -> 1
- net /D_rs: track 58.8 -> 52.8 mm
- net /D_d4: track 75.0 -> 69.1 mm, vias 2 -> 1
- net Net-(D8-K): track 67.2 -> 62.0 mm
- net Net-(D7-K): track 74.2 -> 69.0 mm
- net Net-(D6-K): track 79.3 -> 74.1 mm
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Other:
- board text added: "CybICS v0.2"
- board text removed: "CybICS v0.1"
- board text removed: "GND"
- board text removed: "Matthias Niedermaier"
