File: hardware/pcb/CybICS.kicad_pcb (KiCad board)
At the start: 2 copper layers, 160 x 100 mm, 79 parts, among them J1 Raspberry_Pi_2_3, J2 Conn_01x03_Pin, J3 Conn_01x05_Pin, J4 USB_C_Receptacle_USB2.0, SW1 SW_Push, SW2 SW_Push, SW3 SW_Push, U1 STM32G070RBTx

Commit message: fix(hardware): correct the LED series resistors and the yellow LED part
R1/R2/R4/R6/R10/R21/R23/R25 are drawn as 330R but carried C52548, which
is 0805W8F330LT5E -- 330 mΩ, not 330 Ω. The L in that part code is
Uniroyal's milliohm marker, and both LCSC and JLCPCB's parts database
index it at 0.33 Ω. The six red, two yellow and two blue indicators
were therefore assembled with no effective current limiting: each one
settles at roughly its full rated current against the GPIO's own
impedance, and ten such pins take the STM32G070 past its 100 mA total
I/O budget. Corrected to C17630 (0805W8F3300T5E, 330 Ω), which is also
a basic-library part.

That correction alone would have regressed two colours, because the
0.33 Ω part was the only reason they lit at all:

  - D7/D9 are drawn as LED YELLOW but carried C434441, SZYY1206W -- a
    *white* LED with a yellow lens and Vf 3.1 V. Across a real 330 Ω
    from the 3V3 rail it has ~0.05 V of headroom and stays dark.
    Replaced with C93094 (NCD1206Y1), an actual yellow part with
    Vf 1.6-2.6 V and the same 1206 body.
  - D3/D10 are blue at Vf 2.6-3.1 V, which cannot run off 330 Ω either,
    and no blue LED exists below ~2.6 V. R5 and R8 therefore move to
    100R/C17408 -- the value the nine greens already use, and already a
    basic part -- giving the blues about 3 mA.

All four LED parts keep the existing LED_1210_3225Metric land pattern:
1206 and 1210 share the 3.2 mm terminal span, which is why the 1206
parts already specified here fit.

Verified with kicad-cli 8.0.9: ERC and DRC report 0 violations and 0
unconnected items, and the exported BOM groups R5/R8 with the 100R set
and shows C17630 on the eight remaining 330R positions and C93094 on
D7/D9. Stock and library type were read from LCSC and JLCPCB's parts
database, not from a live quote. Claude has no access to the hardware,
so the resulting currents are calculated from datasheet figures rather
than measured.

Refs #238

Co-Authored-By: Claude Opus 5 (1M context)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
Parts:
- R5, R8: value 330R -> 100R
Changed lines of the file:
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@@
 			)
 		)
-		(property "JLCPCB Part #" "C52548"
+		(property "JLCPCB Part #" "C17630"
 			(at 0 0 0)
 			(layer "F.Fab")
@@
 			)
 		)
-		(property "Value" "330R"
+		(property "Value" "100R"
 			(at 0 1.65 90)
 			(layer "F.Fab")
@@
 			)
 		)
-		(property "JLCPCB Part #" "C52548"
+		(property "JLCPCB Part #" "C17408"
 			(at 199.584252 -10.015748 0)
 			(layer "F.Fab")
@@
 			)
 		)
-		(property "JLCPCB Part #" "C52548"
+		(property "JLCPCB Part #" "C17630"
 			(at 0 0 0)
 			(layer "F.Fab")
@@
 			)
 		)
-		(property "JLCPCB Part #" "C434441"
+		(property "JLCPCB Part #" "C93094"
 			(at 0 0 0)
 			(layer "F.Fab")
@@
 			)
 		)
-		(property "JLCPCB Part #" "C52548"
+		(property "JLCPCB Part #" "C17630"
 			(at 183.584252 5.984252 0)
 			(layer "F.Fab")
@@
 			)
 		)
-		(property "JLCPCB Part #" "C434441"
+		(property "JLCPCB Part #" "C93094"
 			(at 0 0 0)
 			(layer "F.Fab")
@@
 			)
 		)
-		(property "JLCPCB Part #" "C52548"
+		(property "JLCPCB Part #" "C17630"
 			(at 179.584252 9.984252 0)
 			(layer "F.Fab")
@@
 			)
 		)
-		(property "Value" "330R"
+		(property "Value" "100R"
 			(at 0 1.65 90)
 			(layer "F.Fab")
@@
 			)
 		)
-		(property "JLCPCB Part #" "C52548"
+		(property "JLCPCB Part #" "C17408"
 			(at 163.584252 25.984252 0)
 			(layer "F.Fab")
@@
 			)
 		)
-		(property "JLCPCB Part #" "C52548"
+		(property "JLCPCB Part #" "C17630"
 			(at 0 0 0)
 			(layer "F.Fab")
@@
 			)
 		)
-		(property "JLCPCB Part #" "C52548"
+		(property "JLCPCB Part #" "C17630"
 			(at 195.584252 -6.015748 0)
 			(layer "F.Fab")
@@
 			)
 		)
-		(property "JLCPCB Part #" "C52548"
+		(property "JLCPCB Part #" "C17630"
 			(at 187.584252 1.984252 0)
 			(layer "F.Fab")
@@
 			)
 		)
-		(property "JLCPCB Part #" "C52548"
+		(property "JLCPCB Part #" "C17630"
 			(at 171.584252 17.984252 0)
 			(layer "F.Fab")
