File: hardware/pcb/CybICS.kicad_sch (KiCad schematic)
At the start: 75 parts, among them J1 Raspberry_Pi_2_3, J2 Conn_01x03_Pin, J3 Conn_01x05_Pin, SW1 SW_Push, SW2 SW_Push, SW3 SW_Push, U1 STM32G070RBTx

Commit message: chore(hardware): move the 0R and 100nF lines to JLCPCB basic parts
C304192 (0R) and C38141 (100nF) were extended-library parts with basic
equivalents in the same 0805 footprint: C17477 (0805W8F0000T5E) and
C49678 (CC0805KRX7R9BB104), both with millions in stock. JLCPCB charges
a feeder loading fee per unique extended part, so together with the
330R correction in the previous commit this removes three of them from
every build of this board.

Nothing else can move, which is worth recording so the next person does
not go looking:

  - The four LED lines have no basic equivalent in any package. JLCPCB's
    basic library holds two LEDs in total, C84256 (red) and C2297
    (emerald), both 0805 -- so going basic would mean relaying out all
    19 footprints and giving up yellow and blue entirely.
  - The two basic tactile switches are SMD (5.1x5.1 mm and 4x3 mm) and
    do not fit the board's THT SW_PUSH_6mm_H5mm footprint.
  - The STM32, the LCD module, the Pi socket, both pin headers, the
    USB-C receptacle and the potentiometer have no basic parts in their
    categories at all.
  - 100R, 1kR, 10kR, 5.1kR and 4.7uF were already basic.

Verified with kicad-cli 8.0.9: ERC and DRC report 0 violations and 0
unconnected items, and the exported BOM shows C17477 on R13-R19 and
C49678 on C1/C2/C4. Library type and stock come from JLCPCB's parts
database rather than a live quote, so confirm both at checkout.

Co-Authored-By: Claude Opus 5 (1M context) <noreply@anthropic.com>
Claude-Session: https://claude.ai/code/session_011zbigHZaGiZii3etPu8DwT
Parts:
- C1, C2, C4: JLCPCB Part # C38141 -> C49678
- R13, R14, R15, R16, R17, R18, R19: JLCPCB Part # C304192 -> C17477
Changed lines of the file:
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@@
 			)
 		)
-		(property "JLCPCB Part #" "C304192"
+		(property "JLCPCB Part #" "C17477"
 			(at 132.08 44.45 90)
 			(effects
@@
 			)
 		)
-		(property "JLCPCB Part #" "C304192"
+		(property "JLCPCB Part #" "C17477"
 			(at 132.08 77.47 90)
 			(effects
@@
 			)
 		)
-		(property "JLCPCB Part #" "C38141"
+		(property "JLCPCB Part #" "C49678"
 			(at 36.83 30.48 0)
 			(effects
@@
 			)
 		)
-		(property "JLCPCB Part #" "C304192"
+		(property "JLCPCB Part #" "C17477"
 			(at 132.08 80.01 90)
 			(effects
@@
 			)
 		)
-		(property "JLCPCB Part #" "C38141"
+		(property "JLCPCB Part #" "C49678"
 			(at 68.58 27.94 0)
 			(effects
@@
 			)
 		)
-		(property "JLCPCB Part #" "C304192"
+		(property "JLCPCB Part #" "C17477"
 			(at 193.04 52.07 90)
 			(effects
@@
 			)
 		)
-		(property "JLCPCB Part #" "C304192"
+		(property "JLCPCB Part #" "C17477"
 			(at 193.04 54.61 90)
 			(effects
@@
 			)
 		)
-		(property "JLCPCB Part #" "C38141"
+		(property "JLCPCB Part #" "C49678"
 			(at 22.86 48.26 0)
 			(effects
@@
 			)
 		)
-		(property "JLCPCB Part #" "C304192"
+		(property "JLCPCB Part #" "C17477"
 			(at 132.08 57.15 90)
 			(effects
@@
 			)
 		)
-		(property "JLCPCB Part #" "C304192"
+		(property "JLCPCB Part #" "C17477"
 			(at 132.08 46.99 90)
 			(effects
