File: hardware/pcb/CybICS.kicad_sch (KiCad schematic)
At the start: 88 parts, among them J1 Raspberry_Pi_2_3, J2 Conn_01x03_Pin, J3 Conn_01x05_Pin, SW1 SW_Push, SW2 SW_Push, SW3 7*7*5-6P-L WX, U1 STM32G070RBTx

Commit message: fix(hardware): put the LEDs on 0805 footprints and Basic parts
The LEDs sat on 1210 footprints while the ordered parts were 1206 packages.
JLCPCB's own checker flags this -- it is the warning d4ch5 photographed on
issue #238, "Das Footprint (1210) dieses Bauteils stimmt nicht mit dem in
Ihrer BOM angegebenen (1206) ueberein" -- and the issue is still open. Earlier
in this branch the yellow LED was swapped and the footprint moved to the
HandSolder variant, which left the size mismatch untouched; calling that
resolved was wrong.

Fixing it meant choosing a size, and 0805 is the only one where JLCPCB has
Basic LEDs at all: there are exactly four, red C84256, green C2297, yellow
C2296 and white C34499. Nothing is Basic in 1206 or 1210. So the blue LEDs on
D3 "Full" and D10 "Empty" become white -- they mark the two extreme tank
states rather than carrying the red/yellow/green severity meaning, so a
neutral colour suits them, and white's 2.6-3.2 V forward voltage sits in the
same band as blue's 2.6-3.1 V, so the existing 100R series resistors are
unchanged.

All 19 LEDs are now Basic. That drops the unique SMD Extended parts from 8 to
4 -- only the navigation switch, the trimmer, the STM32 and the USB-C socket
remain, and none of those has a Basic equivalent at any package size. At
roughly $3 of feeder fee per unique SMD part, that is about $12 saved per
order regardless of quantity, plus about $0.10 per board on part prices.

Two things the verification caught that a "19 footprints swapped" message
would have hidden. D11, D12 and D13 carry a rotation inside their pad `(at
...)` tokens, which the position rewrite did not match, so they ended up with
0805-sized pads at 1210 positions -- a broken hybrid that showed up as three
silkscreen-over-pad warnings. And D7 had a 0.975 mm track stub that used to
run inside the tall 1210 pad and dangled once the pad shrank; it connected
nothing and was removed.

Verified: kicad-cli DRC from hardware/pcb reports 0 violations, 0 unconnec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
Parts:
- D1, D14, D16, D18, D5, D6: footprint LED_SMD:LED_1210_3225Metric_Pad1.42x2.65mm_HandSolder -> LED_SMD:LED_0805_2012Metric_Pad1.15x1.40mm_HandSolder; JLCPCB Part # C434438 -> C84256
- D10, D3: value LED BLUE -> LED WHITE; footprint LED_SMD:LED_1210_3225Metric_Pad1.42x2.65mm_HandSolder -> LED_SMD:LED_0805_2012Metric_Pad1.15x1.40mm_HandSolder; JLCPCB Part # C434440 -> C34499
- D11, D12, D13, D15, D17, D19, D2, D4, D8: footprint LED_SMD:LED_1210_3225Metric_Pad1.42x2.65mm_HandSolder -> LED_SMD:LED_0805_2012Metric_Pad1.15x1.40mm_HandSolder; JLCPCB Part # C434442 -> C2297
- D7, D9: footprint LED_SMD:LED_1210_3225Metric_Pad1.42x2.65mm_HandSolder -> LED_SMD:LED_0805_2012Metric_Pad1.15x1.40mm_HandSolder; JLCPCB Part # C93094 -> C2296
Changed lines of the file:
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@@
 			)
 		)
-		(property "Footprint" "LED_SMD:LED_1210_3225Metric_Pad1.42x2.65mm_HandSolder"
+		(property "Footprint" "LED_SMD:LED_0805_2012Metric_Pad1.15x1.40mm_HandSolder"
 			(at 99.06 163.83 0)
 			(hide yes)
@@
 			)
 		)
-		(property "JLCPCB Part #" "C434442"
+		(property "JLCPCB Part #" "C2297"
 			(at 99.06 163.83 0)
 			(hide yes)
@@
 			)
 		)
-		(property "Footprint" "LED_SMD:LED_1210_3225Metric_Pad1.42x2.65mm_HandSolder"
+		(property "Footprint" "LED_SMD:LED_0805_2012Metric_Pad1.15x1.40mm_HandSolder"
 			(at 201.93 133.35 0)
 			(hide yes)
@@
 			)
 		)
-		(property "JLCPCB Part #" "C434438"
+		(property "JLCPCB Part #" "C84256"
 			(at 201.93 133.35 0)
 			(hide yes)
@@
 			)
 		)
-		(property "Footprint" "LED_SMD:LED_1210_3225Metric_Pad1.42x2.65mm_HandSolder"
+		(property "Footprint" "LED_SMD:LED_0805_2012Metric_Pad1.15x1.40mm_HandSolder"
 			(at 170.18 132.08 0)
 			(hide yes)
@@
 			)
 		)
-		(property "JLCPCB Part #" "C434442"
+		(property "JLCPCB Part #" "C2297"
 			(at 170.18 132.08 0)
 			(hide yes)
@@
 			)
 		)
-		(property "Value" "LED BLUE"
+		(property "Value" "LED WHITE"
 			(at 168.5925 138.43 0)
 			(show_name no)
@@
 			)
 		)
-		(property "Footprint" "LED_SMD:LED_1210_3225Metric_Pad1.42x2.65mm_HandSolder"
+		(property "Footprint" "LED_SMD:LED_0805_2012Metric_Pad1.15x1.40mm_HandSolder"
 			(at 170.18 142.24 0)
 			(hide yes)
@@
 			)
 		)
-		(property "JLCPCB Part #" "C434440"
+		(property "JLCPCB Part #" "C34499"
 			(at 170.18 142.24 0)
 			(hide yes)
@@
 			)
 		)
-		(property "Footprint" "LED_SMD:LED_1210_3225Metric_Pad1.42x2.65mm_HandSolder"
+		(property "Footprint" "LED_SMD:LED_0805_2012Metric_Pad1.15x1.40mm_HandSolder"
 			(at 243.84 133.35 0)
 			(hide yes)
@@
 			)
 		)
-		(property "JLCPCB Part #" "C434442"
+		(property "JLCPCB Part #" "C2297"
 			(at 243.84 133.35 0)
 			(hide yes)
@@
 			)
 		)
-		(property "Footprint" "LED_SMD:LED_1210_3225Metric_Pad1.42x2.65mm_HandSolder"
+		(property "Footprint" "LED_SMD:LED_0805_2012Metric_Pad1.15x1.40mm_HandSolder"
 			(at 34.29 153.67 0)
 			(hide yes)
@@
 			)
 		)
-		(property "JLCPCB Part #" "C434438"
+		(property "JLCPCB Part #" "C84256"
 			(at 34.29 153.67 0)
 			(hide yes)
@@
 			)
 		)
-		(property "Footprint" "LED_SMD:LED_1210_3225Metric_Pad1.42x2.65mm_HandSolder"
+		(property "Footprint" "LED_SMD:LED_0805_2012Metric_Pad1.15x1.40mm_HandSolder"
 			(at 234.95 157.48 0)
 			(hide yes)
@@
 			)
 		)
-		(property "JLCPCB Part #" "C434442"
+		(property "JLCPCB Part #" "C2297"
 			(at 234.95 157.48 0)
 			(hide yes)
@@
 			)
 		)
-		(property "Footprint" "LED_SMD:LED_1210_3225Metric_Pad1.42x2.65mm_HandSolder"
+		(property "Footprint" "LED_SMD:LED_0805_2012Metric_Pad1.15x1.40mm_HandSolder"
 			(at 135.89 132.08 0)
 			(hide yes)
@@
 			)
 		)
-		(property "JLCPCB Part #" "C93094"
+		(property "JLCPCB Part #" "C2296"
 			(at 135.89 132.08 0)
 			(hide yes)
@@
 			)
 		)
-		(property "Footprint" "LED_SMD:LED_1210_3225Metric_Pad1.42x2.65mm_HandSolder"
+		(property "Footprint" "LED_SMD:LED_0805_2012Metric_Pad1.15x1.40mm_HandSolder"
 			(at 243.84 146.05 0)
 			(hide yes)
@@
 			)
 		)
-		(property "JLCPCB Part #" "C434442"
+		(property "JLCPCB Part #" "C2297"
 			(at 243.84 146.05 0)
 			(hide yes)
@@
 			)
 		)
-		(property "Footprint" "LED_SMD:LED_1210_3225Metric_Pad1.42x2.65mm_HandSolder"
+		(property "Footprint" "LED_SMD:LED_0805_2012Metric_Pad1.15x1.40mm_HandSolder"
 			(at 67.31 163.83 0)
 			(hide yes)
@@
 			)
 		)
-		(property "JLCPCB Part #" "C434442"
+		(property "JLCPCB Part #" "C2297"
 			(at 67.31 163.83 0)
 			(hide yes)
@@
 			)
 		)
-		(property "Footprint" "LED_SMD:LED_1210_3225Metric_Pad1.42x2.65mm_HandSolder"
+		(property "Footprint" "LED_SMD:LED_0805_2012Metric_Pad1.15x1.40mm_HandSolder"
 			(at 135.89 120.65 0)
 			(hide yes)
@@
 			)
 		)
-		(property "JLCPCB Part #" "C434438"
+		(property "JLCPCB Part #" "C84256"
 			(at 135.89 120.65 0)
 			(hide yes)
@@
 			)
 		)
-		(property "Footprint" "LED_SMD:LED_1210_3225Metric_Pad1.42x2.65mm_HandSolder"
+		(property "Footprint" "LED_SMD:LED_0805_2012Metric_Pad1.15x1.40mm_HandSolder"
 			(at 135.89 154.94 0)
 			(hide yes)
@@
 			)
 		)
-		(property "JLCPCB Part #" "C93094"
+		(property "JLCPCB Part #" "C2296"
 			(at 135.89 154.94 0)
 			(hide yes)
@@
 			)
 		)
-		(property "Footprint" "LED_SMD:LED_1210_3225Metric_Pad1.42x2.65mm_HandSolder"
+		(property "Footprint" "LED_SMD:LED_0805_2012Metric_Pad1.15x1.40mm_HandSolder"
 			(at 99.06 153.67 0)
 			(hide yes)
@@
 			)
 		)
-		(property "JLCPCB Part #" "C434438"
+		(property "JLCPCB Part #" "C84256"
 			(at 99.06 153.67 0)
 			(hide yes)
@@
 			)
 		)
-		(property "Footprint" "LED_SMD:LED_1210_3225Metric_Pad1.42x2.65mm_HandSolder"
+		(property "Footprint" "LED_SMD:LED_0805_2012Metric_Pad1.15x1.40mm_HandSolder"
 			(at 170.18 121.92 0)
 			(hide yes)
@@
 			)
 		)
-		(property "JLCPCB Part #" "C434438"
+		(property "JLCPCB Part #" "C84256"
 			(at 170.18 121.92 0)
 			(hide yes)
@@
 			)
 		)
-		(property "Footprint" "LED_SMD:LED_1210_3225Metric_Pad1.42x2.65mm_HandSolder"
+		(property "Footprint" "LED_SMD:LED_0805_2012Metric_Pad1.15x1.40mm_HandSolder"
 			(at 135.89 143.51 0)
 			(hide yes)
@@
 			)
 		)
-		(property "JLCPCB Part #" "C434442"
+		(property "JLCPCB Part #" "C2297"
 			(at 135.89 143.51 0)
 			(hide yes)
@@
 			)
 		)
-		(property "Footprint" "LED_SMD:LED_1210_3225Metric_Pad1.42x2.65mm_HandSolder"
+		(property "Footprint" "LED_SMD:LED_0805_2012Metric_Pad1.15x1.40mm_HandSolder"
 			(at 34.29 163.83 0)
 			(hide yes)
@@
 			)
 		)
-		(property "JLCPCB Part #" "C434442"
+		(property "JLCPCB Part #" "C2297"
 			(at 34.29 163.83 0)
 			(hide yes)
@@
 			)
 		)
-		(property "Footprint" "LED_SMD:LED_1210_3225Metric_Pad1.42x2.65mm_HandSolder"
+		(property "Footprint" "LED_SMD:LED_0805_2012Metric_Pad1.15x1.40mm_HandSolder"
 			(at 67.31 153.67 0)
 			(hide yes)
@@
 			)
 		)
-		(property "JLCPCB Part #" "C434438"
+		(property "JLCPCB Part #" "C84256"
 			(at 67.31 153.67 0)
 			(hide yes)
@@
 			)
 		)
-		(property "Footprint" "LED_SMD:LED_1210_3225Metric_Pad1.42x2.65mm_HandSolder"
+		(property "Footprint" "LED_SMD:LED_0805_2012Metric_Pad1.15x1.40mm_HandSolder"
 			(at 201.93 121.92 0)
 			(hide yes)
@@
 			)
 		)
-		(property "JLCPCB Part #" "C434442"
+		(property "JLCPCB Part #" "C2297"
 			(at 201.93 121.92 0)
 			(hide yes)
@@
 			)
 		)
-		(property "Value" "LED BLUE"
+		(property "Value" "LED WHITE"
 			(at 134.3025 162.56 0)
 			(show_name no)
@@
 			)
 		)
-		(property "Footprint" "LED_SMD:LED_1210_3225Metric_Pad1.42x2.65mm_HandSolder"
+		(property "Footprint" "LED_SMD:LED_0805_2012Metric_Pad1.15x1.40mm_HandSolder"
 			(at 135.89 166.37 0)
 			(hide yes)
@@
 			)
 		)
-		(property "JLCPCB Part #" "C434440"
+		(property "JLCPCB Part #" "C34499"
 			(at 135.89 166.37 0)
 			(hide yes)

Commit message: fix(hardware): rebalance the green LEDs after the Basic swap
The Basic green C2297 is far more efficient than the part it replaced: 430 mcd
at 5 mA against 70 mcd at 20 mA. Left on its 100R series resistor it would have
drawn 4.5 mA and put out around 390 mcd, roughly fourteen times the red and
yellow indicators. On a board where red means "Critical" and green means
"Normal", that is the wrong way round.

The nine green LEDs each have their own resistor, so they move from 100R to 1k
on their own: R3, R7, R9, R11, R12, R20, R22, R24 and R26. R5 and R8 stay at
100R because they feed the two white LEDs, whose forward voltage is a volt
higher.

1k is already on the board sixteen times, so this adds no BOM line -- C17513
goes from 16 to 25 placements and C17408 drops from 11 to 2.

The result is 39 mcd green, 56 white, 28 red and 25 yellow, a spread of 2.2x
instead of 14x. Green lands where it already is today: the outgoing part
managed about 42 mcd on its 100R, so the green indicators will look unchanged
rather than dimmer. The 0.45 mA figure is conservative -- forward voltage at
that current sits below the 5 mA typical, so the real current and brightness
will be somewhat higher.

Verified: kicad-cli DRC from hardware/pcb reports 0 violations, 0 unconnected
items and 0 schematic parity issues. Only values and part numbers changed; the
0805 resistor footprints and all routing are untouched.

Co-Authored-By: Claude Opus 5 (1M context) <noreply@anthropic.com>
Claude-Session: https://claude.ai/code/session_011zbigHZaGiZii3etPu8DwT
Parts:
- R11, R12, R20, R22, R24, R26, R3, R7, R9: value 100R -> 1kR; JLCPCB Part # C17408 -> C17513
Changed lines of the file:
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@@
 			)
 		)
-		(property "Value" "100R"
+		(property "Value" "1kR"
 			(at 233.68 129.54 90)
 			(show_name no)
@@
 			)
 		)
-		(property "JLCPCB Part #" "C17408"
+		(property "JLCPCB Part #" "C17513"
 			(at 233.68 133.35 90)
 			(hide yes)
@@
 			)
 		)
-		(property "Value" "100R"
+		(property "Value" "1kR"
 			(at 57.15 160.02 90)
 			(show_name no)
@@
 			)
 		)
-		(property "JLCPCB Part #" "C17408"
+		(property "JLCPCB Part #" "C17513"
 			(at 57.15 163.83 90)
 			(hide yes)
@@
 			)
 		)
-		(property "Value" "100R"
+		(property "Value" "1kR"
 			(at 125.73 139.7 90)
 			(show_name no)
@@
 			)
 		)
-		(property "JLCPCB Part #" "C17408"
+		(property "JLCPCB Part #" "C17513"
 			(at 125.73 143.51 90)
 			(hide yes)
@@
 			)
 		)
-		(property "Value" "100R"
+		(property "Value" "1kR"
 			(at 88.9 160.02 90)
 			(show_name no)
@@
 			)
 		)
-		(property "JLCPCB Part #" "C17408"
+		(property "JLCPCB Part #" "C17513"
 			(at 88.9 163.83 90)
 			(hide yes)
@@
 			)
 		)
-		(property "Value" "100R"
+		(property "Value" "1kR"
 			(at 160.02 128.27 90)
 			(show_name no)
@@
 			)
 		)
-		(property "JLCPCB Part #" "C17408"
+		(property "JLCPCB Part #" "C17513"
 			(at 160.02 132.08 90)
 			(hide yes)
@@
 			)
 		)
-		(property "Value" "100R"
+		(property "Value" "1kR"
 			(at 24.13 160.02 90)
 			(show_name no)
@@
 			)
 		)
-		(property "JLCPCB Part #" "C17408"
+		(property "JLCPCB Part #" "C17513"
 			(at 24.13 163.83 90)
 			(hide yes)
@@
 			)
 		)
-		(property "Value" "100R"
+		(property "Value" "1kR"
 			(at 224.79 153.67 90)
 			(show_name no)
@@
 			)
 		)
-		(property "JLCPCB Part #" "C17408"
+		(property "JLCPCB Part #" "C17513"
 			(at 224.79 157.48 90)
 			(hide yes)
@@
 			)
 		)
-		(property "Value" "100R"
+		(property "Value" "1kR"
 			(at 191.77 118.11 90)
 			(show_name no)
@@
 			)
 		)
-		(property "JLCPCB Part #" "C17408"
+		(property "JLCPCB Part #" "C17513"
 			(at 191.77 121.92 90)
 			(hide yes)
@@
 			)
 		)
-		(property "Value" "100R"
+		(property "Value" "1kR"
 			(at 233.68 142.24 90)
 			(show_name no)
@@
 			)
 		)
-		(property "JLCPCB Part #" "C17408"
+		(property "JLCPCB Part #" "C17513"
 			(at 233.68 146.05 90)
 			(hide yes)

Commit message: chore(hardware): drop the Amphenol header on J2 for a CJT A2541WV-3P
J2 carried C168677, an Amphenol ICC 68000-103HLF, at $0.2813 per board
against $0.0658 for C5445396 (CJT A2541WV-3P) -- a factor of four on a
three-pin 2.54 mm header with no property that earns it. J3 already uses
A2541WV-5P, so this also puts both service headers in one family: the
UART header gains the same keyed housing the SWD header has, which is
worth having on a board where students plug into both.

Both parts stay Extended, and that costs nothing here. The $3.07 feeder
loading fee applies to Extended parts that go onto a pick-and-place
feeder; a through-hole part is hand soldered instead, at $3.58 per order
plus $0.0164 per joint, with no per-type fee. So the whole saving is part
price: $0.22 per board, and the BOM keeps the same number of lines.

Checked against the fee-free library before settling for a cheaper
Extended part rather than a Basic one: JLCPCB's Basic library holds 351
parts and the Preferred Extended tier, which is also exempt from the
feeder fee, holds 1235. Neither contains a single connector -- the
categories Pin Headers, Female Headers and USB Connectors have zero
fee-free parts between them. There is no Basic header to move to.

The footprint is unchanged, so the pad pattern is identical. The
A2541WV's shroud does overhang the 8.65 x 3.60 mm courtyard by about a
millimetre a side, which is the same situation J3 has had all along:
nothing is near enough to care, the closest part is R25 at 12.4 mm and
DS1's outline starts at x=130.05 while J2 ends at 118.65.

Verified with kicad-cli 10.0.6: DRC with --refill-zones reports 0
violations, 0 unconnected items and 0 schematic parity issues; ERC
--severity-error reports 0; the exported BOM shows C5445396 on J2 and
C225480 still on J3; the position export carries 79 SMD rows and no FID
lines. Prices and library type were read from JLCPCB's parts database,
not from a live quote, so confirm both at checkout.

Bare DRC without --r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
Parts:
- J2: JLCPCB Part # C168677 -> C5445396
Changed lines of the file:
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@@
 			)
 		)
-		(property "JLCPCB Part #" "C168677"
+		(property "JLCPCB Part #" "C5445396"
 			(at 267.97 130.81 0)
 			(hide yes)
